File: logic_signal_amp.kicad_pcb (KiCad board)
At the start: 2 copper layers, 43.5 x 34 mm, 10 parts, among them J1 Conn_01x05_Pin, J2 Conn_01x10_Pin, Q1 AO3400A, Q2 AO3400A, Q3 AO3400A, Q4 AO3400A

Commit message: final PCB
Routing:
- net +12V: track 0.00 -> 20.6 mm
- net GND: track 12.7 -> 29.4 mm, vias 0 -> 10
- added copper zone on B.Cu, net GND
